Commit message: adding hokuyo and nav2

File: leo_description/urdf/macros.xacro (robot description, xacro)
@@ -1,4 +1,5 @@
 <?xml version="1.0" encoding="utf-8"?>
 <robot xmlns:xacro="http://www.ros.org/wiki/xacro">
+  <xacro:include filename="$(find leo_description)/urdf/sensors/all_sensors.urdf.xacro" />
   <xacro:macro name="leo"
                params="default_antenna:=true
@@ -9,4 +10,7 @@
                        imu_translation:='0.0628 -0.0314 -0.0393'
                        mecanum_wheels:=false">
+    <xacro:sensor_hokuyo prefix="${link_prefix}front_laser" parent="${link_prefix}base_link">
+        <origin xyz="0.105 0.0 0.05" rpy="0 0 0"/>
+    </xacro:sensor_hokuyo>
     <xacro:macro name="rocker_link" params="name">
       <link name="${link_prefix}rocker_${name}_link">

Commit message: adding asus xtion camera

File: leo_description/urdf/macros.xacro (robot description, xacro)
@@ -11,6 +11,32 @@
                        mecanum_wheels:=false">
     <xacro:sensor_hokuyo prefix="${link_prefix}front_laser" parent="${link_prefix}base_link">
-        <origin xyz="0.105 0.0 0.05" rpy="0 0 0"/>
+      <origin xyz="0.105 0.0 0.05" rpy="0 0 0"/>
     </xacro:sensor_hokuyo>
+    <link name="camera_mast_link">
+      <visual>
+        <origin rpy="0 0 0" xyz="0 0 0" />
+        <geometry>
+          <box size="0.025 0.025 1.2"/>
+        </geometry>
+      </visual>
+      <collision>
+        <origin rpy="0 0 0" xyz="0 0 0" />
+        <geometry>
+          <box size="0.025 0.025 1.2"/>
+        </geometry>
+      </collision>
+      <!-- <xacro:solid_cuboid_inertial
+                rpy="0 0 0" xyz="0 0 0"
+                mass="1"
+                x="0.1" y="0.1" z="1.2" /> -->
+    </link>
+    <joint name="camera_mast_link_joint" type="fixed">
+      <origin rpy="0 0 0" xyz="0.0 0.0 0.6"/>
+      <parent link="${link_prefix}base_link" />
+      <child link="camera_mast_link" />
+    </joint>
+    <xacro:sensor_asus_xtion prefix="asus_camera" parent="camera_mast_link">
+      <origin xyz="0.04 0.0 0.58" rpy="0 ${pi/4} 0"/>
+    </xacro:sensor_asus_xtion>
     <xacro:macro name="rocker_link" params="name">
       <link name="${link_prefix}rocker_${name}_link">
@@ -428,34 +454,34 @@
     <gazebo reference="${link_prefix}camera_frame">
       <sensor name="camera" type="camera">
-          <camera name="leo_camera">
-              <horizontal_fov>1.9</horizontal_fov>
-              <image>
-                  <width>640</width>
-                  <height>480</height>
-                  <format>R8G8B8</format>
-              </image>
-              <clip>
-                  <near>0.2</near>
-                  <far>300</far>
-              </clip>
-              <noise>
-                <type>gaussian</type>
-                <mean>0.0</mean>
-                <stddev>0.007</stddev>
-              </noise>
-              <distortion>
-                <k1>-0.279817</k1>
-                <k2>0.060321</k2>
-                <k3>0.000487</k3>
-                <p1>0.000310</p1>
-                <p2>0.000000</p2>
-                <center>0.5 0.5</center>
-              </distortion>
-          </camera>
-          <always_on>1</always_on>
-          <update_rate>30</update_rate>
-          <visualize>true</visualize>
-          <topic>${link_prefix}camera/image_raw</topic>
-          <ignition_frame_id>${link_prefix}camera_frame</ignition_frame_id>
+        <camera name="leo_camera">
+          <horizontal_fov>1.9</horizontal_fov>
+          <image>
+            <width>640</width>
+            <height>480</height>
+            <format>R8G8B8</format>
+          </image>
+          <clip>
+            <near>0.2</near>
+            <far>300</far>
+          </clip>
+          <noise>
+            <type>gaussian</type>
+            <mean>0.0</mean>
+            <stddev>0.007</stddev>
+          </noise>
+          <distortion>
+            <k1>-0.279817</k1>
+            <k2>0.060321</k2>
+            <k3>0.000487</k3>
+            <p1>0.000310</p1>
+            <p2>0.000000</p2>
+            <center>0.5 0.5</center>
+          </distortion>
+        </camera>
+        <always_on>1</always_on>
+        <update_rate>30</update_rate>
+        <visualize>true</visualize>
+        <topic>${link_prefix}camera/image_raw</topic>
+        <ignition_frame_id>${link_prefix}camera_frame</ignition_frame_id>
       </sensor>
     </gazebo>

File: leo_description/urdf/sensors/all_sensors.urdf.xacro (robot description, xacro)
@@ -22,3 +22,4 @@
   <xacro:include filename="$(find leo_description)/urdf/sensors/hokuyo.urdf.xacro" />
   <!-- Camera -->
+  <xacro:include filename="$(find leo_description)/urdf/sensors/asus_xtion.urdf.xacro" />
 </robot>

Commit message: fixing camera position

File: leo_description/urdf/macros.xacro (robot description, xacro)
@@ -23,5 +23,5 @@
         <origin rpy="0 0 0" xyz="0 0 0" />
         <geometry>
-          <box size="0.025 0.025 1.2"/>
+          <box size="0.03 0.03 1.2"/>
         </geometry>
       </collision>
@@ -37,5 +37,5 @@
     </joint>
     <xacro:sensor_asus_xtion prefix="asus_camera" parent="camera_mast_link">
-      <origin xyz="0.04 0.0 0.58" rpy="0 ${pi/4} 0"/>
+      <origin xyz="0.045 0.0 0.57" rpy="0 ${pi/4} 0"/>
     </xacro:sensor_asus_xtion>
     <xacro:macro name="rocker_link" params="name">
